File: C64 Pi1541-III Module Panel/C64 Pi1541-III Module Panel.kicad_pcb (KiCad board)
At the start: 2 copper layers, 100 x 23.2 mm, 15 parts, among them IC1 OLED, J1 Module Panel, M1 Mounting_Pin, M2 Mounting_Pin, M3 Mounting_Pin, M4 Mounting_Pin, SW1 BACK, SW2 INSERT

Commit message: ...
Other:
- net class Default removed
- net class PWR removed
