File: faceplates/C64 Pi1541-III Module FP1/C64 Pi1541-III Module FP1.kicad_pcb (KiCad board)
At the start: 2 copper layers, 100 x 35 mm, 9 parts, among them M1 Mounting_Pin, M2 Mounting_Pin, M3 Mounting_Pin, M4 Mounting_Pin

Commit message: ...
Other:
- net class Default removed
- net class PWR removed
